Commit message: Unit 4: 4.4.1   Move a laser up and down by position

File: my_box_bot_description/urdf/box_bot_control_complete.urdf (robot description, URDF)
Before this commit: robot box_bot, 10 links, 9 joints
Links:
- added link laser_scan_frame
- added link laser_scan_link, mass 0.01; collision box size=0.074986 0.074935 0.0408; visual mesh filename=package://my_box_bot_description/meshes/sensors/rplidar.dae scale=1.0 1.0 1.0
Joints:
- added joint laser_scan_frame_joint: type fixed, parent laser_scan_link, child laser_scan_frame, origin xyz=0 0 0.03 rpy=0 0 0, axis 0 0 0
- added joint laser_scan_link_joint: type prismatic, parent chassis, child laser_scan_link, origin xyz=0.0 0.0 0.05 rpy=0 0 0, axis 0 0 1, limit lower=-0.1 upper=0.0 effort=20.0 velocity=2.0
